Commit message: 添加控制节点

File: engineer_description/urdf/exchanger/engineer_exchanger.urdf.xacro (robot description, xacro)
@@ -7,11 +7,4 @@
   <!-- Import plugin -->
   <xacro:include filename="$(find engineer_description)/urdf/exchanger/engineer_exchanger_plugin.gazebo"/>
-  <link name="world"/>
-  <joint name="world_ebase_joint" type="fixed">
-    <origin rpy="0 0 0" xyz="0 0 0"/>
-    <parent link="world"/>
-    <child link="ebase_link"/>
-    <axis xyz="0 0 0"/>
-  </joint>
   <link name="ebase_link">
     <visual>
@@ -32,6 +25,6 @@
     <inertial>
       <origin rpy="0 0 0" xyz="0 0 0.01"/>
-      <mass value="32"/>
-      <inertia ixx="2.66773" ixy="0" ixz="0" iyy="2.66773" iyz="0" izz="5.33333"/>
+      <mass value="3200"/>
+      <inertia ixx="266.773" ixy="0" ixz="0" iyy="266.773" iyz="0" izz="533.333"/>
     </inertial>
   </link>
@@ -121,7 +114,7 @@
       </geometry>
       <material>
-        <ambient>0 0 0 1</ambient>
-        <diffuse>0 0 0 1</diffuse>
-        <specular>0 0 0 0</specular>
+        <ambient>1 0 0 1</ambient>
+        <diffuse>1 0 0 1</diffuse>
+        <specular>1 0 0 0</specular>
         <emissive>1 0 0 1</emissive>
       </material>

File: engineer_description/urdf/robot/engineer_robot.urdf.xacro (robot description, xacro)
@@ -41,5 +41,5 @@
   </link>
   <xacro:engineer_wheel_LF prefix="LF" parent="base_link" origin_x="0.20286" origin_y="0.2023" origin_z="-0.012411" rotation_x="-1.5708"/>
-  <xacro:engineer_roller prefix="roller_LF_1" parent="wheel_LF" origin_z="${roller_origin_z1}" rotation_x="${roller_rotation_x1}" rotation_z="${roller_rotation_z1}"/>
+  <!-- <xacro:engineer_roller prefix="roller_LF_1" parent="wheel_LF" origin_z="${roller_origin_z1}" rotation_x="${roller_rotation_x1}" rotation_z="${roller_rotation_z1}"/>
   <xacro:engineer_roller prefix="roller_LF_2" parent="wheel_LF" origin_z="${roller_origin_z1}" rotation_x="${roller_rotation_x1}" rotation_z="${roller_rotation_z2}"/>
   <xacro:engineer_roller prefix="roller_LF_3" parent="wheel_LF" origin_z="${roller_origin_z1}" rotation_x="${roller_rotation_x1}" rotation_z="${roller_rotation_z3}"/>
@@ -56,7 +56,7 @@
   <xacro:engineer_roller prefix="roller_LF_14" parent="wheel_LF" origin_z="${roller_origin_z1}" rotation_x="${roller_rotation_x1}" rotation_z="${roller_rotation_z14}"/>
   <xacro:engineer_roller prefix="roller_LF_15" parent="wheel_LF" origin_z="${roller_origin_z1}" rotation_x="${roller_rotation_x1}" rotation_z="${roller_rotation_z15}"/>
-  <xacro:engineer_roller prefix="roller_LF_16" parent="wheel_LF" origin_z="${roller_origin_z1}" rotation_x="${roller_rotation_x1}" rotation_z="${roller_rotation_z16}"/>
+  <xacro:engineer_roller prefix="roller_LF_16" parent="wheel_LF" origin_z="${roller_origin_z1}" rotation_x="${roller_rotation_x1}" rotation_z="${roller_rotation_z16}"/> -->
   <xacro:engineer_wheel_RF prefix="RF" parent="base_link" origin_x="0.20286" origin_y="-0.2023" origin_z="-0.012411" rotation_x="-1.5708"/>
-  <xacro:engineer_roller prefix="roller_RF_1" parent="wheel_RF" origin_z="${roller_origin_z2}" rotation_x="${roller_rotation_x2}" rotation_z="${roller_rotation_z1}"/>
+  <!-- <xacro:engineer_roller prefix="roller_RF_1" parent="wheel_RF" origin_z="${roller_origin_z2}" rotation_x="${roller_rotation_x2}" rotation_z="${roller_rotation_z1}"/>
   <xacro:engineer_roller prefix="roller_RF_2" parent="wheel_RF" origin_z="${roller_origin_z2}" rotation_x="${roller_rotation_x2}" rotation_z="${roller_rotation_z2}"/>
   <xacro:engineer_roller prefix="roller_RF_3" parent="wheel_RF" origin_z="${roller_origin_z2}" rotation_x="${roller_rotation_x2}" rotation_z="${roller_rotation_z3}"/>
@@ -73,7 +73,7 @@
   <xacro:engineer_roller prefix="roller_RF_14" parent="wheel_RF" origin_z="${roller_origin_z2}" rotation_x="${roller_rotation_x2}" rotation_z="${roller_rotation_z14}"/>
   <xacro:engineer_roller prefix="roller_RF_15" parent="wheel_RF" origin_z="${roller_origin_z2}" rotation_x="${roller_rotation_x2}" rotation_z="${roller_rotation_z15}"/>
-  <xacro:engineer_roller prefix="roller_RF_16" parent="wheel_RF" origin_z="${roller_origin_z2}" rotation_x="${roller_rotation_x2}" rotation_z="${roller_rotation_z16}"/>
+  <xacro:engineer_roller prefix="roller_RF_16" parent="wheel_RF" origin_z="${roller_origin_z2}" rotation_x="${roller_rotation_x2}" rotation_z="${roller_rotation_z16}"/> -->
   <xacro:engineer_wheel_RB prefix="RB" parent="base_link" origin_x="-0.20286" origin_y="-0.2023" origin_z="-0.012411" rotation_x="-1.5708"/>
-  <xacro:engineer_roller prefix="roller_RB_1" parent="wheel_RB" origin_z="${roller_origin_z1}" rotation_x="${roller_rotation_x1}" rotation_z="${roller_rotation_z1}"/>
+  <!-- <xacro:engineer_roller prefix="roller_RB_1" parent="wheel_RB" origin_z="${roller_origin_z1}" rotation_x="${roller_rotation_x1}" rotation_z="${roller_rotation_z1}"/>
   <xacro:engineer_roller prefix="roller_RB_2" parent="wheel_RB" origin_z="${roller_origin_z1}" rotation_x="${roller_rotation_x1}" rotation_z="${roller_rotation_z2}"/>
   <xacro:engineer_roller prefix="roller_RB_3" parent="wheel_RB" origin_z="${roller_origin_z1}" rotation_x="${roller_rotation_x1}" rotation_z="${roller_rotation_z3}"/>
@@ -90,7 +90,7 @@
   <xacro:engineer_roller prefix="roller_RB_14" parent="wheel_RB" origin_z="${roller_origin_z1}" rotation_x="${roller_rotation_x1}" rotation_z="${roller_rotation_z14}"/>
   <xacro:engineer_roller prefix="roller_RB_15" parent="wheel_RB" origin_z="${roller_origin_z1}" rotation_x="${roller_rotation_x1}" rotation_z="${roller_rotation_z15}"/>
-  <xacro:engineer_roller prefix="roller_RB_16" parent="wheel_RB" origin_z="${roller_origin_z1}" rotation_x="${roller_rotation_x1}" rotation_z="${roller_rotation_z16}"/>
+  <xacro:engineer_roller prefix="roller_RB_16" parent="wheel_RB" origin_z="${roller_origin_z1}" rotation_x="${roller_rotation_x1}" rotation_z="${roller_rotation_z16}"/> -->
   <xacro:engineer_wheel_LB prefix="LB" parent="base_link" origin_x="-0.20286" origin_y="0.2023" origin_z="-0.012411" rotation_x="-1.5708"/>
-  <xacro:engineer_roller prefix="roller_LB_1" parent="wheel_LB" origin_z="${roller_origin_z2}" rotation_x="${roller_rotation_x2}" rotation_z="${roller_rotation_z1}"/>
+  <!-- <xacro:engineer_roller prefix="roller_LB_1" parent="wheel_LB" origin_z="${roller_origin_z2}" rotation_x="${roller_rotation_x2}" rotation_z="${roller_rotation_z1}"/>
   <xacro:engineer_roller prefix="roller_LB_2" parent="wheel_LB" origin_z="${roller_origin_z2}" rotation_x="${roller_rotation_x2}" rotation_z="${roller_rotation_z2}"/>
   <xacro:engineer_roller prefix="roller_LB_3" parent="wheel_LB" origin_z="${roller_origin_z2}" rotation_x="${roller_rotation_x2}" rotation_z="${roller_rotation_z3}"/>
@@ -107,5 +107,5 @@
   <xacro:engineer_roller prefix="roller_LB_14" parent="wheel_LB" origin_z="${roller_origin_z2}" rotation_x="${roller_rotation_x2}" rotation_z="${roller_rotation_z14}"/>
   <xacro:engineer_roller prefix="roller_LB_15" parent="wheel_LB" origin_z="${roller_origin_z2}" rotation_x="${roller_rotation_x2}" rotation_z="${roller_rotation_z15}"/>
-  <xacro:engineer_roller prefix="roller_LB_16" parent="wheel_LB" origin_z="${roller_origin_z2}" rotation_x="${roller_rotation_x2}" rotation_z="${roller_rotation_z16}"/>
+  <xacro:engineer_roller prefix="roller_LB_16" parent="wheel_LB" origin_z="${roller_origin_z2}" rotation_x="${roller_rotation_x2}" rotation_z="${roller_rotation_z16}"/> -->
   <xacro:engineer_boom prefix="link1" parent="base_link" joint_origin="${link1_joint}" limit="${link1_limits}"
                        inertial_origin="${link1_inertial}" mass="${link1_mass}" inertia="${link1_inertia}"/>
@@ -122,4 +122,29 @@
   <xacro:engineer_boom prefix="link7" parent="link6" joint_origin="${link7_joint}" limit="${link7_limits}"
                        inertial_origin="${link7_inertial}" mass="${link7_mass}" inertia="${link7_inertia}"/>
+  <joint name="gripper_joint" type="fixed">
+    <origin xyz="0 0 0.019" rpy="0 0 0"/>
+    <parent link="link7"/>
+    <child link="gripper_link"/>
+  </joint>
+  <link name="gripper_link">
+    <inertial>
+      <origin xyz="0 0 0" rpy="0 0 0"/>
+      <mass value="0.001"/>
+      <inertia ixx="1.6E-09" ixy="0" ixz="0"
+               iyy="1.6E-09" iyz="0" izz="1.6E-08"/>
+    </inertial>
+    <visual>
+      <origin xyz="0 0 0" rpy="0 0 0"/>
+      <geometry>
+        <box size="0.001 0.001 0.001" />
+      </geometry>
+    </visual>
+    <collision>
+      <origin xyz="0 0 0" rpy="0 0 0"/>
+      <geometry>
+        <box size="0.001 0.001 0.001" />
+      </geometry>
+    </collision>
+  </link>
   <xacro:engineer_little_arm prefix="left_z" parent="base_link" joint_type="prismatic" joint_origin="${left_z_joint}" joint_axis="${left_z_axis}"
                              limit="${left_z_limits}" inertial_origin="${left_z_inertial}" mass="${left_z_mass}" inertia="${left_z_inertia}"/>
@@ -134,5 +159,5 @@
   <xacro:engineer_little_arm prefix="right_yaw" parent="right_x_link" joint_type="revolute" joint_origin="${right_yaw_joint}" joint_axis="${right_yaw_axis}"
                              limit="${right_yaw_limits}" inertial_origin="${right_yaw_inertial}" mass="${right_yaw_mass}" inertia="${right_yaw_inertia}"/>
-  <xacro:engineer_depth_camera prefix="engineer_depth_camera" parent="link4" origin_x="0" origin_y="0" origin_z="0.075" rotation_x="0" rotation_y="0" rotation_z="0"/>
+  <xacro:engineer_depth_camera prefix="engineer_depth_camera" parent="link3" origin_x="0.152" origin_y="-0.078" origin_z="0.0" rotation_x="1.5708" rotation_y="0" rotation_z="0"/>
   <!-- Wheel Trans -->
   <xacro:engineer_wheel_trans prefix="LF"/>
@@ -141,10 +166,90 @@
   <xacro:engineer_wheel_trans prefix="LB"/>
   <!-- Wheel Gazebo -->
-  <xacro:engineer_wheel_gazebo prefix="LF"/>
+  <!-- <xacro:engineer_wheel_gazebo prefix="LF"/>
   <xacro:engineer_wheel_gazebo prefix="RF"/>
   <xacro:engineer_wheel_gazebo prefix="RB"/>
-  <xacro:engineer_wheel_gazebo prefix="LB"/>
+  <xacro:engineer_wheel_gazebo prefix="LB"/> -->
+  <gazebo reference="wheel_LF">
+    <selfCollide>true</selfCollide>
+    <gravity>true</gravity>
+    <!-- <mu1>50</mu1>
+    <mu2>50</mu2> -->
+    <collision>
+      <surface>
+        <friction>
+          <ode>
+            <mu>50.0</mu>
+            <mu2>0.0</mu2>
+            <fdir1>1 -1 0</fdir1>
+          </ode>
+        </friction>
+      </surface>
+    </collision>
+    <kp>1e50</kp>
+    <kd>1e50</kd>
+    <material>Gazebo/White</material>
+  </gazebo>
+  <gazebo reference="wheel_RF">
+    <selfCollide>true</selfCollide>
+    <gravity>true</gravity>
+    <!-- <mu1>50</mu1>
+    <mu2>50</mu2> -->
+    <collision>
+      <surface>
+        <friction>
+          <ode>
+            <mu>50.0</mu>
+            <mu2>0.0</mu2>
+            <fdir1>1 1 0</fdir1>
+          </ode>
+        </friction>
+      </surface>
+    </collision>
+    <kp>1e50</kp>
+    <kd>1e50</kd>
+    <material>Gazebo/White</material>
+  </gazebo>
+  <gazebo reference="wheel_RB">
+    <selfCollide>true</selfCollide>
+    <gravity>true</gravity>
+    <!-- <mu1>50</mu1>
+    <mu2>50</mu2> -->
+    <collision>
+      <surface>
+        <friction>
+          <ode>
+            <mu>50.0</mu>
+            <mu2>0.0</mu2>
+            <fdir1>1 -1 0</fdir1>
+          </ode>
+        </friction>
+      </surface>
+    </collision>
+    <kp>1e50</kp>
+    <kd>1e50</kd>
+    <material>Gazebo/White</material>
+  </gazebo>
+  <gazebo reference="wheel_LB">
+    <selfCollide>true</selfCollide>
+    <gravity>true</gravity>
+    <!-- <mu1>50</mu1>
+    <mu2>50</mu2> -->
+    <collision>
+      <surface>
+        <friction>
+          <ode>
+            <mu>50.0</mu>
+            <mu2>0.0</mu2>
+            <fdir1>1 1 0</fdir1>
+          </ode>
+        </friction>
+      </surface>
+    </collision>
+    <kp>1e50</kp>
+    <kd>1e50</kd>
+    <material>Gazebo/White</material>
+  </gazebo>
   <!-- Roller Gazebo -->
-  <xacro:engineer_roller_gazebo prefix="roller_LF_1"/>
+  <!-- <xacro:engineer_roller_gazebo prefix="roller_LF_1"/>
   <xacro:engineer_roller_gazebo prefix="roller_LF_2"/>
   <xacro:engineer_roller_gazebo prefix="roller_LF_3"/>
@@ -209,5 +314,5 @@
   <xacro:engineer_roller_gazebo prefix="roller_LB_14"/>
   <xacro:engineer_roller_gazebo prefix="roller_LB_15"/>
-  <xacro:engineer_roller_gazebo prefix="roller_LB_16"/>
+  <xacro:engineer_roller_gazebo prefix="roller_LB_16"/> -->
   <!-- Arm Gazebo -->
   <xacro:engineer_arm_gazebo prefix="base_link"/>
@@ -219,4 +324,11 @@
   <xacro:engineer_arm_gazebo prefix="link6"/>
   <xacro:engineer_arm_gazebo prefix="link7"/>
+  <gazebo reference="gripper_link">
+    <mu1>50</mu1>
+    <mu2>50</mu2>
+    <material>Gazebo/Grey</material>
+    <self_collide>true</self_collide>
+    <gravity>true</gravity>
+  </gazebo>
   <xacro:engineer_arm_gazebo prefix="left_z_link"/>
   <xacro:engineer_arm_gazebo prefix="left_x_link"/>

File: engineer_description/urdf/robot/engineer_wheel_LB.urdf.xacro (robot description, xacro)
@@ -15,5 +15,5 @@
         <origin xyz="0 0 0" rpy="0 0 0" />
         <geometry>
-          <mesh filename="file://$(find engineer_description)/meshes/left-threaded_mecanum_wheel_wheel.STL" />
+          <mesh filename="file://$(find engineer_description)/meshes/wheel_LB.STL" />
         </geometry>
         <material name="white">
@@ -24,6 +24,15 @@
         <origin xyz="0 0 0" rpy="0 0 0" />
         <geometry>
-          <mesh filename="file://$(find engineer_description)/meshes/left-threaded_mecanum_wheel_wheel.STL" />
+          <mesh filename="file://$(find engineer_description)/meshes/wheel_LB.STL" />
         </geometry>
+        <surface>
+          <friction>
+            <ode>
+              <mu>1.0</mu>
+              <mu2>0.0</mu2>
+              <fdir1>1 1 0</fdir1>
+            </ode>
+          </friction>
+        </surface>
       </collision>
       <inertial>

File: engineer_description/urdf/robot/engineer_wheel_LF.urdf.xacro (robot description, xacro)
@@ -15,5 +15,5 @@
         <origin xyz="0 0 0" rpy="0 0 0" />
         <geometry>
-          <mesh filename="file://$(find engineer_description)/meshes/right-threaded_mecanum_wheel_wheel.STL" />
+          <mesh filename="file://$(find engineer_description)/meshes/wheel_LF.STL" />
         </geometry>
         <material name="white">
@@ -24,6 +24,15 @@
         <origin xyz="0 0 0" rpy="0 0 0" />
         <geometry>
-          <mesh filename="file://$(find engineer_description)/meshes/right-threaded_mecanum_wheel_wheel.STL" />
+          <mesh filename="file://$(find engineer_description)/meshes/wheel_LF.STL" />
         </geometry>
+        <surface>
+          <friction>
+            <ode>
+              <mu>1.0</mu>
+              <mu2>0.0</mu2>
+              <fdir1>1 -1 0</fdir1>
+            </ode>
+          </friction>
+        </surface>
       </collision>
       <inertial>

File: engineer_description/urdf/robot/engineer_wheel_RB.urdf.xacro (robot description, xacro)
@@ -15,5 +15,5 @@
         <origin xyz="0 0 0" rpy="0 0 0" />
         <geometry>
-          <mesh filename="file://$(find engineer_description)/meshes/right-threaded_mecanum_wheel_wheel.STL" />
+          <mesh filename="file://$(find engineer_description)/meshes/wheel_RB.STL" />
         </geometry>
         <material name="white">
@@ -24,6 +24,15 @@
         <origin xyz="0 0 0" rpy="0 0 0" />
         <geometry>
-          <mesh filename="file://$(find engineer_description)/meshes/right-threaded_mecanum_wheel_wheel.STL" />
+          <mesh filename="file://$(find engineer_description)/meshes/wheel_RB.STL" />
         </geometry>
+        <surface>
+          <friction>
+            <ode>
+              <mu>1.0</mu>
+              <mu2>0.0</mu2>
+              <fdir1>1 -1 0</fdir1>
+            </ode>
+          </friction>
+        </surface>
       </collision>
       <inertial>

File: engineer_description/urdf/robot/engineer_wheel_RF.urdf.xacro (robot description, xacro)
@@ -15,5 +15,5 @@
         <origin xyz="0 0 0" rpy="0 0 0" />
         <geometry>
-          <mesh filename="file://$(find engineer_description)/meshes/left-threaded_mecanum_wheel_wheel.STL" />
+          <mesh filename="file://$(find engineer_description)/meshes/wheel_RF.STL" />
         </geometry>
         <material name="white">
@@ -24,6 +24,15 @@
         <origin xyz="0 0 0" rpy="0 0 0" />
         <geometry>
-          <mesh filename="file://$(find engineer_description)/meshes/left-threaded_mecanum_wheel_wheel.STL" />
+          <mesh filename="file://$(find engineer_description)/meshes/wheel_RF.STL" />
         </geometry>
+        <surface>
+          <friction>
+            <ode>
+              <mu>1.0</mu>
+              <mu2>0.0</mu2>
+              <fdir1>1 1 0</fdir1>
+            </ode>
+          </friction>
+        </surface>
       </collision>
       <inertial>

Commit message: 优化模型

File: engineer_description/urdf/exchanger/engineer_exchanger.urdf.xacro (robot description, xacro)
@@ -1,9 +1,6 @@
 <?xml version="1.0"?>
 <robot xmlns:xacro="http://www.ros.org/wiki/xacro" name="exchanger">
-  <!-- Import parameters -->
   <xacro:include filename="$(find engineer_description)/urdf/exchanger/engineer_exchanger_parameters.xacro" />
-  <!-- Import arm -->
   <xacro:include filename="$(find engineer_description)/urdf/exchanger/engineer_exchanger_arm.urdf.xacro"/>
-  <!-- Import plugin -->
   <xacro:include filename="$(find engineer_description)/urdf/exchanger/engineer_exchanger_plugin.gazebo"/>
   <link name="ebase_link">
@@ -48,7 +45,7 @@
     </inertial>
     <visual>
-      <origin xyz="0 0 0" rpy="0 0 0" />
+      <origin rpy="0 -1.5708 0" xyz="0 0 -0.24"/>
       <geometry>
-        <mesh filename="file://$(find engineer_description)/meshes/ore.STL" />
+        <mesh filename="file://$(find engineer_description)/meshes/collision/ore.STL" />
       </geometry>
       <material name="">
@@ -57,12 +54,12 @@
     </visual>
     <collision>
-      <origin xyz="0 0 0" rpy="0 0 0" />
+      <origin rpy="0 -1.5708 0" xyz="0 0 -0.24"/>
       <geometry>
-        <mesh filename="file://$(find engineer_description)/meshes/ore.STL" />
+        <mesh filename="file://$(find engineer_description)/meshes/collision/ore.STL" />
       </geometry>
     </collision>
   </link>
   <joint name="ore_joint" type="fixed">
-    <origin xyz="0 0 0.025" rpy="0 -1.5708 0" />
+    <origin xyz="0 0 0" rpy="0 0 0" />
     <parent link="elink6" />
     <child link="ore" />
@@ -76,7 +73,7 @@
     </inertial>
     <visual>
-      <origin xyz="0 0 0" rpy="0 0 0" />
+      <origin rpy="0 -1.5708 0" xyz="0 0 0"/>
       <geometry>
-        <mesh filename="file://$(find engineer_description)/meshes/light.STL" />
+        <mesh filename="file://$(find engineer_description)/meshes/collision/light.STL" />
       </geometry>
       <material name="">
@@ -86,12 +83,12 @@
     </visual>
     <collision>
-      <origin xyz="0 0 0" rpy="0 0 0" />
+      <origin rpy="0 -1.5708 0" xyz="0 0 0"/>
       <geometry>
-        <mesh filename="file://$(find engineer_description)/meshes/light.STL" />
+        <mesh filename="file://$(find engineer_description)/meshes/collision/light.STL" />
       </geometry>
     </collision>
   </link>
   <joint name="light_joint" type="fixed">
-    <origin xyz="0.24 0 0" rpy="0 0 0" />
+    <origin xyz="0 0 0" rpy="0 0 0" />
     <parent link="ore" />
     <child link="light" />
@@ -114,5 +111,5 @@
       </geometry>
       <material>
-        <ambient>1 0 0 1</ambient>
+        <ambient>1 1 1 1</ambient>
         <diffuse>1 0 0 1</diffuse>
         <specular>1 0 0 0</specular>

File: engineer_description/urdf/exchanger/engineer_exchanger_parameters.xacro (robot description, xacro)
@@ -32,7 +32,7 @@
   <xacro:property name="elink5_inertial" value="${[-0.05, -0.05, 3.13E-19]}"/>
   <!-- link6参数 -->
-  <xacro:property name="elink6_joint" value="${[0.05, -0.125, 0, 1.5708, 0, 0]}"/>
+  <xacro:property name="elink6_joint" value="${[0.05, -0.39, 0, 1.5708, 0, 0]}"/>
   <xacro:property name="elink6_limits" value="${[-1.5708, 1.5708]}"/>
-  <xacro:property name="elink6_link" value="${[0, 0, 0, 0, 0, 0]}"/>
+  <xacro:property name="elink6_link" value="${[0, 0, -0.265, 0, 0, 0]}"/>
   <xacro:property name="elink6_inertial" value="${[-6.1756E-16, 3.0762E-16, 0.14137]}"/>
 </robot>
