Commit message: 优化模型

File: engineer_description/urdf/robot/engineer_wheel.urdf.xacro (robot description, xacro)
@@ -3,33 +3,37 @@
   <xacro:include filename="$(find engineer_description)/urdf/robot/engineer_wheel.gazebo"/>
   <xacro:include filename="$(find engineer_description)/urdf/robot/engineer_wheel.transmission.xacro"/>
-  <xacro:macro name="engineer_wheel" params="prefix parent origin_x origin_y origin_z rotation_x">
+  <xacro:macro name="engineer_wheel" params="prefix params">
     <joint name="${prefix}_joint" type="continuous">
-      <parent link="${parent}"/>
+      <parent link="base_link"/>
       <child link="wheel_${prefix}"/>
-      <origin xyz="${origin_x} ${origin_y} ${origin_z}" rpy="${rotation_x} 0 0"/>
+      <origin xyz="${params.joint[0]} ${params.joint[1]} ${params.joint[2]}" rpy="${params.joint[3]} ${params.joint[4]} ${params.joint[5]}"/>
       <axis xyz="0 0 1"/>
-      <!-- <dynamics damping="4.0" friction="5.0"/> -->
     </joint>
     <link name="wheel_${prefix}">
       <visual>
-        <origin xyz="0 0 0" rpy="0 0 0" />
         <geometry>
-          <mesh filename="file://$(find engineer_description)/meshes/wheel_${prefix}.STL" />
+          <mesh filename="file://$(find engineer_description)/meshes/collision/wheel_${prefix}.STL" />
         </geometry>
-        <material name="white">
-          <color rgba="1.0 1.0 1.0 1.0"/>
-        </material>
       </visual>
       <collision>
         <origin xyz="0 0 0" rpy="0 0 0" />
         <geometry>
-          <mesh filename="file://$(find engineer_description)/meshes/wheel_${prefix}.STL" />
+          <sphere radius="0.077" />
         </geometry>
+        <surface>
+          <friction>
+            <ode>
+              <mu>1.0</mu>
+              <mu2>1.0</mu2>
+              <fdir1>${params.fdir1}</fdir1>
+            </ode>
+          </friction>
+        </surface>
       </collision>
       <inertial>
         <origin xyz="0 0 0" rpy="0 0 0" />
-        <mass value="0.192661" />
-        <inertia ixx="0.000408" ixy="0" ixz="0"
-                 iyy="0.000408" iyz="0" izz="0.00078" />
+        <mass value="0.007056" />
+        <inertia ixx="0.000017" ixy="0" ixz="0"
+                 iyy="0.000017" iyz="0" izz="0.000033" />
       </inertial>
     </link>
